File: hardware/pack-monitor.kicad_pcb (KiCad board)
At the start: 2 copper layers, 100 x 50 mm, 12 parts, among them J1 1985302, Q1 PMOS, SW1 RESET_BTN, U1 Pico, U2 TSR 0.5-2450

Commit message: Update pmos pins
Parts:
- moved Q1 4.32 mm to (191.7, 86.7)
Connections:
- Q1 pad 1: Net-(Q1-D) -> /VBUS
- Q1 pad 2: /VBUS -> /VSYS
- Q1 pad 3: /VSYS -> Net-(Q1-D)
Routing:
- net /VSYS: track 64.6 -> 57.9 mm
- net /VBUS: track 63.5 -> 66.8 mm
- net Net-(Q1-D): track 15.7 -> 14.5 mm
Changed lines of the file:
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@@
 			(solder_mask_margin 0.102)
 		)
+		(model "${KIPRJMOD}/libraries/1985302.stp"
+			(offset
+				(xyz 1.5 0 0)
+			)
+			(scale
+				(xyz 1 1 1)
+			)
+			(rotate
+				(xyz 0 0 0)
+			)
+		)
 	)
 	(footprint "Button_Switch_THT:SW_PUSH_6mm"
@@
 	(footprint "Package_TO_SOT_SMD:TSOT-23_HandSoldering"
 		(layer "F.Cu")
-		(at 194.5 90)
+		(at 191.72 86.6975)
 		(descr "5-pin TSOT23 package, http://cds.linear.com/docs/en/packaging/SOT_5_05-08-1635.pdf")
 		(tags "TSOT-23 Hand-soldering")
@@
 			)
 		)
-		(property "Sim.Pins" "1=D 2=G 3=S"
+		(property "Sim.Pins" "1=G 2=S 3=D"
 			(at 0 0 0)
 			(unlocked yes)
@@
 			(layers "F.Cu" "F.Paste" "F.Mask")
 			(roundrect_rratio 0.25)
-			(net 13 "Net-(Q1-D)")
-			(pinfunction "D")
-			(pintype "passive")
+			(net 15 "/VBUS")
+			(pinfunction "G")
+			(pintype "input")
 		)
 		(pad "2" smd roundrect
@@
 			(layers "F.Cu" "F.Paste" "F.Mask")
 			(roundrect_rratio 0.25)
-			(net 15 "/VBUS")
-			(pinfunction "G")
-			(pintype "input")
+			(net 14 "/VSYS")
+			(pinfunction "S")
+			(pintype "passive")
 		)
 		(pad "3" smd roundrect
@@
 			(layers "F.Cu" "F.Paste" "F.Mask")
 			(roundrect_rratio 0.25)
-			(net 14 "/VSYS")
-			(pinfunction "S")
+			(net 13 "Net-(Q1-D)")
+			(pinfunction "D")
 			(pintype "passive")
 		)
@@
 	)
 	(segment
-		(start 197.37 89.05)
-		(end 204.4625 81.9575)
+		(start 193.43 86.6975)
+		(end 198.6425 86.6975)
 		(width 0.2)
 		(layer "F.Cu")
@@
 	)
 	(segment
-		(start 192.79 89.05)
-		(end 197.37 89.05)
+		(start 204.4625 81.9575)
+		(end 204.4625 80.8775)
 		(width 0.2)
 		(layer "F.Cu")
@@
 	)
 	(segment
-		(start 204.4625 81.9575)
+		(start 198.6425 86.6975)
 		(end 204.4625 80.8775)
 		(width 0.2)
@@
 	)
 	(segment
-		(start 183 86.5)
-		(end 135.5 86.5)
+		(start 187.4575 87.6475)
+		(end 186.47 86.66)
 		(width 0.2)
 		(layer "F.Cu")
@@
 	)
 	(segment
-		(start 135.5 86.5)
-		(end 134.48 85.48)
+		(start 136.11 86.66)
+		(end 134.25 84.8)
+		(width 0.2)
+		(layer "F.Cu")
+		(net 14)
+	)
+	(segment
+		(start 190.01 87.6475)
+		(end 187.4575 87.6475)
 		(width 0.2)
 		(layer "F.Cu")
@@
 	)
 	(segment
-		(start 186.5 90)
-		(end 196.21 90)
+		(start 186.47 86.66)
+		(end 136.11 86.66)
 		(width 0.2)
 		(layer "F.Cu")
@@
 	)
 	(segment
-		(start 183 86.5)
-		(end 186.5 90)
+		(start 183.74 87.37)
+		(end 134.28 87.37)
 		(width 0.2)
 		(layer "F.Cu")
-		(net 14)
+		(net 15)
+	)
+	(segment
+		(start 191.88 87.6175)
+		(end 191.88 88.99)
+		(width 0.2)
+		(layer "F.Cu")
+		(net 15)
+	)
+	(segment
+		(start 134.28 87.37)
+		(end 131.71 84.8)
+		(width 0.2)
+		(layer "F.Cu")
+		(net 15)
 	)
 	(segment
-		(start 186.79 90.95)
-		(end 192.79 90.95)
+		(start 190.81 90.06)
+		(end 186.43 90.06)
 		(width 0.2)
 		(layer "F.Cu")
@@
 	)
 	(segment
-		(start 131.94 84.5)
-		(end 134.44 87)
+		(start 186.43 90.06)
+		(end 183.74 87.37)
 		(width 0.2)
 		(layer "F.Cu")
@@
 	)
 	(segment
-		(start 134.44 87)
-		(end 182.84 87)
+		(start 190.01 85.7475)
+		(end 191.88 87.6175)
 		(width 0.2)
 		(layer "F.Cu")
@@
 	)
 	(segment
-		(start 182.84 87)
-		(end 186.79 90.95)
+		(start 191.88 88.99)
+		(end 190.81 90.06)
 		(width 0.2)
 		(layer "F.Cu")
