File: hardware/pack-monitor.kicad_sch (KiCad schematic)
At the start: 12 parts, among them J1 1985302, Q1 PMOS, SW1 RESET_BTN, U1 Pico, U2 TSR 0.5-2450

Commit message: Update pmos pins
Connections:
- net VBUS: now also Q1.1 (G); no longer Q1.2 (G)
- net VSYS: now also Q1.2 (S); no longer Q1.3 (S)
- net at U2.3 (OUT): now also Q1.3 (D); no longer Q1.1 (D)
Changed lines of the file:
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@@
 			)
 		)
-		(property "Sim.Pins" "1=D 2=G 3=S"
+		(property "Sim.Pins" "1=G 2=S 3=D"
 			(at 99.06 129.54 0)
 			(effects
